Commit message: use gzserver replace gazebo

File: src/ylr1d_mid_control/urdf/ylr1d_mid.xacro (robot description, xacro)
@@ -1,5 +1,4 @@
 <?xml version="1.0" encoding="utf-8"?>
-<robot xmlns:xacro="http://wiki.ros.org/xacro"
-       name="ylr1d">
+<robot xmlns:xacro="http://wiki.ros.org/xacro" name="ylr1d">
   <!-- ============================================ -->
   <!-- YAML config values (links.yaml, colors.yaml,  -->
@@ -8,4 +7,13 @@
   <!-- ============================================ -->
   <xacro:macro name="ylr1d" params="prefix">
+<!-- 添加空的虚拟连接 -->
+<!--
+<link name="${prefix}base_footprint" />
+<joint name="${prefix}base_footprint_joint" type="fixed">
+    <origin xyz="0 0 0.3" rpy="0 0 0" />
+    <parent link="${prefix}base_footprint" />
+    <child link="${prefix}Link_Base" />
+</joint>
+-->
 <link name="${prefix}Link_Base">
     <inertial>
