Commit message: fix model

File: src/ylr1d_description/urdf/ylr1d.urdf (robot description, URDF)
Before this commit: robot ylr1d, 40 links, 39 joints
Joints:
- removed joint Joint_Body2_RightArm1
- added joint Joint_Body2_to_RightArm1: type revolute, parent Link_Body2, child Link_RightArm1, origin xyz=0 0 0.133799999999997 rpy=1.5707963267949 0 0, axis 0 0 1, limit lower=-2.62 upper=2.62 effort=1000.0 velocity=2.83

File: src/ylr1d_description/urdf/ylr1d.xacro (robot description, xacro)
@@ -741,12 +741,12 @@
     </collision>
   </link>
-  <joint name="${prefix}Joint_Body2_RightArm1" type="revolute">
+  <joint name="${prefix}Joint_Body2_to_RightArm1" type="revolute">
     <origin xyz="0 0 0.133799999999997" rpy="1.5707963267949 0 0"/>
     <parent link="Link_Body2"/>
     <child link="Link_RightArm1"/>
     <axis xyz="0 0 1"/>
-    <limit lower="${limits.Joint_Body2_RightArm1.lower}" upper="${limits.Joint_Body2_RightArm1.upper}" effort="${limits.Joint_Body2_RightArm1.effort}" velocity="${limits.Joint_Body2_RightArm1.velocity}"/>
-    <calibration rising="${calibration.Joint_Body2_RightArm1.rising}" falling="${calibration.Joint_Body2_RightArm1.falling}"/>
-    <dynamics damping="${dynamics.Joint_Body2_RightArm1.damping}" friction="${dynamics.Joint_Body2_RightArm1.friction}"/>
+    <limit lower="${limits.Joint_Body2_to_RightArm1.lower}" upper="${limits.Joint_Body2_to_RightArm1.upper}" effort="${limits.Joint_Body2_to_RightArm1.effort}" velocity="${limits.Joint_Body2_to_RightArm1.velocity}"/>
+    <calibration rising="${calibration.Joint_Body2_to_RightArm1.rising}" falling="${calibration.Joint_Body2_to_RightArm1.falling}"/>
+    <dynamics damping="${dynamics.Joint_Body2_to_RightArm1.damping}" friction="${dynamics.Joint_Body2_to_RightArm1.friction}"/>
   </joint>
   <link name="${prefix}Link_RightArm2">

File: src/ylr1d_description/urdf/ylr1d_gazebo.urdf (robot description, URDF)
Before this commit: robot ylr1d, 40 links, 39 joints
Joints:
- removed joint Joint_Body2_RightArm1
- added joint Joint_Body2_to_RightArm1: type revolute, parent Link_Body2, child Link_RightArm1, origin xyz=0 0 0.133799999999997 rpy=1.5707963267949 0 0, axis 0 0 1, limit lower=-2.62 upper=2.62 effort=1000.0 velocity=2.83

File: src/ylr1d_description/urdf/ylr1d_gazebo.xacro (robot description, xacro)
@@ -741,12 +741,12 @@
     </collision>
   </link>
-  <joint name="${prefix}Joint_Body2_RightArm1" type="revolute">
+  <joint name="${prefix}Joint_Body2_to_RightArm1" type="revolute">
     <origin xyz="0 0 0.133799999999997" rpy="1.5707963267949 0 0"/>
     <parent link="Link_Body2"/>
     <child link="Link_RightArm1"/>
     <axis xyz="0 0 1"/>
-    <limit lower="${limits.Joint_Body2_RightArm1.lower}" upper="${limits.Joint_Body2_RightArm1.upper}" effort="${limits.Joint_Body2_RightArm1.effort}" velocity="${limits.Joint_Body2_RightArm1.velocity}"/>
-    <calibration rising="${calibration.Joint_Body2_RightArm1.rising}" falling="${calibration.Joint_Body2_RightArm1.falling}"/>
-    <dynamics damping="${dynamics.Joint_Body2_RightArm1.damping}" friction="${dynamics.Joint_Body2_RightArm1.friction}"/>
+    <limit lower="${limits.Joint_Body2_to_RightArm1.lower}" upper="${limits.Joint_Body2_to_RightArm1.upper}" effort="${limits.Joint_Body2_to_RightArm1.effort}" velocity="${limits.Joint_Body2_to_RightArm1.velocity}"/>
+    <calibration rising="${calibration.Joint_Body2_to_RightArm1.rising}" falling="${calibration.Joint_Body2_to_RightArm1.falling}"/>
+    <dynamics damping="${dynamics.Joint_Body2_to_RightArm1.damping}" friction="${dynamics.Joint_Body2_to_RightArm1.friction}"/>
   </joint>
   <link name="${prefix}Link_RightArm2">

File: src/ylr1d_mid_control/urdf/ylr1d_mid.xacro (robot description, xacro)
@@ -738,12 +738,12 @@
     </collision>
   </link>
-  <joint name="${prefix}Joint_Body2_RightArm1" type="revolute">
+  <joint name="${prefix}Joint_Body2_to_RightArm1" type="revolute">
     <origin xyz="0 0 0.133799999999997" rpy="1.5707963267949 0 0"/>
     <parent link="Link_Body2"/>
     <child link="Link_RightArm1"/>
     <axis xyz="0 0 1"/>
-    <limit lower="${limits.Joint_Body2_RightArm1.lower}" upper="${limits.Joint_Body2_RightArm1.upper}" effort="${limits.Joint_Body2_RightArm1.effort}" velocity="${limits.Joint_Body2_RightArm1.velocity}"/>
-    <calibration rising="${calibration.Joint_Body2_RightArm1.rising}" falling="${calibration.Joint_Body2_RightArm1.falling}"/>
-    <dynamics damping="${dynamics.Joint_Body2_RightArm1.damping}" friction="${dynamics.Joint_Body2_RightArm1.friction}"/>
+    <limit lower="${limits.Joint_Body2_to_RightArm1.lower}" upper="${limits.Joint_Body2_to_RightArm1.upper}" effort="${limits.Joint_Body2_to_RightArm1.effort}" velocity="${limits.Joint_Body2_to_RightArm1.velocity}"/>
+    <calibration rising="${calibration.Joint_Body2_to_RightArm1.rising}" falling="${calibration.Joint_Body2_to_RightArm1.falling}"/>
+    <dynamics damping="${dynamics.Joint_Body2_to_RightArm1.damping}" friction="${dynamics.Joint_Body2_to_RightArm1.friction}"/>
   </joint>
   <link name="${prefix}Link_RightArm2">
@@ -1666,5 +1666,5 @@
     </joint>
     <!-- Right arm: 7-DOF + 2 fingers (position command) -->
-    <joint name="Joint_Body2_RightArm1">
+    <joint name="Joint_Body2_to_RightArm1">
       <command_interface name="position"/>
       <state_interface name="position"/>
