Commit message: fix the model axis

File: src/ylr1d_description/urdf/ylr1d.urdf (robot description, URDF)
Before this commit: robot ylr1d, 40 links, 39 joints
Joints:
- joint Joint_LBWheelF_to_LBWheel: limit lower=0 upper=0 effort=0 velocity=0 -> (none)

File: src/ylr1d_description/urdf/ylr1d.xacro (robot description, xacro)
@@ -159,5 +159,5 @@
     <parent link="Link_LFWheelF"/>
     <child link="Link_LFWheel"/>
-    <axis xyz="0 0 1"/>
+    <axis xyz="0 0 -1"/>
     <calibration rising="${calibration.Joint_LFWheelF_to_LFWheel.rising}" falling="${calibration.Joint_LFWheelF_to_LFWheel.falling}"/>
     <dynamics damping="${dynamics.Joint_LFWheelF_to_LFWheel.damping}" friction="${dynamics.Joint_LFWheelF_to_LFWheel.friction}"/>
@@ -281,6 +281,5 @@
     <parent link="Link_LBWheelF"/>
     <child link="Link_LBWheel"/>
-    <axis xyz="0 0 1"/>
-    <limit lower="${limits.Joint_LBWheelF_to_LBWheel.lower}" upper="${limits.Joint_LBWheelF_to_LBWheel.upper}" effort="${limits.Joint_LBWheelF_to_LBWheel.effort}" velocity="${limits.Joint_LBWheelF_to_LBWheel.velocity}"/>
+    <axis xyz="0 0 -1"/>
     <calibration rising="${calibration.Joint_LBWheelF_to_LBWheel.rising}" falling="${calibration.Joint_LBWheelF_to_LBWheel.falling}"/>
     <dynamics damping="${dynamics.Joint_LBWheelF_to_LBWheel.damping}" friction="${dynamics.Joint_LBWheelF_to_LBWheel.friction}"/>
@@ -451,5 +450,5 @@
     <parent link="Link_Body2"/>
     <child link="Link_LeftArm1"/>
-    <axis xyz="0 0 -1"/>
+    <axis xyz="0 0 1"/>
     <limit lower="${limits.Joint_Body2_to_LeftArm1.lower}" upper="${limits.Joint_Body2_to_LeftArm1.upper}" effort="${limits.Joint_Body2_to_LeftArm1.effort}" velocity="${limits.Joint_Body2_to_LeftArm1.velocity}"/>
     <calibration rising="${calibration.Joint_Body2_to_LeftArm1.rising}" falling="${calibration.Joint_Body2_to_LeftArm1.falling}"/>
@@ -513,5 +512,5 @@
     <parent link="Link_LeftArm2"/>
     <child link="Link_LeftArm3"/>
-    <axis xyz="0 -1 0"/>
+    <axis xyz="0 1 0"/>
     <limit lower="${limits.Joint_LeftArm2_to_LeftArm3.lower}" upper="${limits.Joint_LeftArm2_to_LeftArm3.upper}" effort="${limits.Joint_LeftArm2_to_LeftArm3.effort}" velocity="${limits.Joint_LeftArm2_to_LeftArm3.velocity}"/>
     <calibration rising="${calibration.Joint_LeftArm2_to_LeftArm3.rising}" falling="${calibration.Joint_LeftArm2_to_LeftArm3.falling}"/>
@@ -544,5 +543,5 @@
     <parent link="Link_LeftArm3"/>
     <child link="Link_LeftArm4"/>
-    <axis xyz="0 0 1"/>
+    <axis xyz="0 0 -1"/>
     <limit lower="${limits.Joint_LeftArm3_to_LeftArm4.lower}" upper="${limits.Joint_LeftArm3_to_LeftArm4.upper}" effort="${limits.Joint_LeftArm3_to_LeftArm4.effort}" velocity="${limits.Joint_LeftArm3_to_LeftArm4.velocity}"/>
     <calibration rising="${calibration.Joint_LeftArm3_to_LeftArm4.rising}" falling="${calibration.Joint_LeftArm3_to_LeftArm4.falling}"/>
@@ -606,5 +605,5 @@
     <parent link="Link_LeftArm5"/>
     <child link="Link_LeftArm6"/>
-    <axis xyz="0 0 1"/>
+    <axis xyz="0 0 -1"/>
     <limit lower="${limits.Joint_LeftArm5_to_LeftArm6.lower}" upper="${limits.Joint_LeftArm5_to_LeftArm6.upper}" effort="${limits.Joint_LeftArm5_to_LeftArm6.effort}" velocity="${limits.Joint_LeftArm5_to_LeftArm6.velocity}"/>
     <calibration rising="${calibration.Joint_LeftArm5_to_LeftArm6.rising}" falling="${calibration.Joint_LeftArm5_to_LeftArm6.falling}"/>
@@ -637,5 +636,5 @@
     <parent link="Link_LeftArm6"/>
     <child link="Link_LeftArm7"/>
-    <axis xyz="0 0 -1"/>
+    <axis xyz="0 0 1"/>
     <limit lower="${limits.Joint_LeftArm6_to_LeftArm7.lower}" upper="${limits.Joint_LeftArm6_to_LeftArm7.upper}" effort="${limits.Joint_LeftArm6_to_LeftArm7.effort}" velocity="${limits.Joint_LeftArm6_to_LeftArm7.velocity}"/>
     <calibration rising="${calibration.Joint_LeftArm6_to_LeftArm7.rising}" falling="${calibration.Joint_LeftArm6_to_LeftArm7.falling}"/>
@@ -745,5 +744,5 @@
     <parent link="Link_Body2"/>
     <child link="Link_RightArm1"/>
-    <axis xyz="0 0 1"/>
+    <axis xyz="0 0 -1"/>
     <limit lower="${limits.Joint_Body2_to_RightArm1.lower}" upper="${limits.Joint_Body2_to_RightArm1.upper}" effort="${limits.Joint_Body2_to_RightArm1.effort}" velocity="${limits.Joint_Body2_to_RightArm1.velocity}"/>
     <calibration rising="${calibration.Joint_Body2_to_RightArm1.rising}" falling="${calibration.Joint_Body2_to_RightArm1.falling}"/>
@@ -838,5 +837,5 @@
     <parent link="Link_RightArm3"/>
     <child link="Link_RightArm4"/>
-    <axis xyz="0 0 -1"/>
+    <axis xyz="0 0 1"/>
     <limit lower="${limits.Joint_RightArm3_to_RightArm4.lower}" upper="${limits.Joint_RightArm3_to_RightArm4.upper}" effort="${limits.Joint_RightArm3_to_RightArm4.effort}" velocity="${limits.Joint_RightArm3_to_RightArm4.velocity}"/>
     <calibration rising="${calibration.Joint_RightArm3_to_RightArm4.rising}" falling="${calibration.Joint_RightArm3_to_RightArm4.falling}"/>
@@ -869,5 +868,5 @@
     <parent link="Link_RightArm4"/>
     <child link="Link_RightArm5"/>
-    <axis xyz="0 0 1"/>
+    <axis xyz="0 0 -1"/>
     <limit lower="${limits.Joint_RightArm4_to_RightArm5.lower}" upper="${limits.Joint_RightArm4_to_RightArm5.upper}" effort="${limits.Joint_RightArm4_to_RightArm5.effort}" velocity="${limits.Joint_RightArm4_to_RightArm5.velocity}"/>
     <calibration rising="${calibration.Joint_RightArm4_to_RightArm5.rising}" falling="${calibration.Joint_RightArm4_to_RightArm5.falling}"/>
@@ -900,5 +899,5 @@
     <parent link="Link_RightArm5"/>
     <child link="Link_RightArm6"/>
-    <axis xyz="0 0 -1"/>
+    <axis xyz="0 0 1"/>
     <limit lower="${limits.Joint_RightArm5_to_RightArm6.lower}" upper="${limits.Joint_RightArm5_to_RightArm6.upper}" effort="${limits.Joint_RightArm5_to_RightArm6.effort}" velocity="${limits.Joint_RightArm5_to_RightArm6.velocity}"/>
     <calibration rising="${calibration.Joint_RightArm5_to_RightArm6.rising}" falling="${calibration.Joint_RightArm5_to_RightArm6.falling}"/>

File: src/ylr1d_description/urdf/ylr1d_gazebo.urdf (robot description, URDF)
Before this commit: robot ylr1d, 40 links, 39 joints
Joints:
- joint Joint_LBWheelF_to_LBWheel: limit lower=0 upper=0 effort=0 velocity=0 -> (none)

File: src/ylr1d_description/urdf/ylr1d_gazebo.xacro (robot description, xacro)
@@ -159,5 +159,5 @@
     <parent link="Link_LFWheelF"/>
     <child link="Link_LFWheel"/>
-    <axis xyz="0 0 1"/>
+    <axis xyz="0 0 -1"/>
     <calibration rising="${calibration.Joint_LFWheelF_to_LFWheel.rising}" falling="${calibration.Joint_LFWheelF_to_LFWheel.falling}"/>
     <dynamics damping="${dynamics.Joint_LFWheelF_to_LFWheel.damping}" friction="${dynamics.Joint_LFWheelF_to_LFWheel.friction}"/>
@@ -281,6 +281,5 @@
     <parent link="Link_LBWheelF"/>
     <child link="Link_LBWheel"/>
-    <axis xyz="0 0 1"/>
-    <limit lower="${limits.Joint_LBWheelF_to_LBWheel.lower}" upper="${limits.Joint_LBWheelF_to_LBWheel.upper}" effort="${limits.Joint_LBWheelF_to_LBWheel.effort}" velocity="${limits.Joint_LBWheelF_to_LBWheel.velocity}"/>
+    <axis xyz="0 0 -1"/>
     <calibration rising="${calibration.Joint_LBWheelF_to_LBWheel.rising}" falling="${calibration.Joint_LBWheelF_to_LBWheel.falling}"/>
     <dynamics damping="${dynamics.Joint_LBWheelF_to_LBWheel.damping}" friction="${dynamics.Joint_LBWheelF_to_LBWheel.friction}"/>
@@ -451,5 +450,5 @@
     <parent link="Link_Body2"/>
     <child link="Link_LeftArm1"/>
-    <axis xyz="0 0 -1"/>
+    <axis xyz="0 0 1"/>
     <limit lower="${limits.Joint_Body2_to_LeftArm1.lower}" upper="${limits.Joint_Body2_to_LeftArm1.upper}" effort="${limits.Joint_Body2_to_LeftArm1.effort}" velocity="${limits.Joint_Body2_to_LeftArm1.velocity}"/>
     <calibration rising="${calibration.Joint_Body2_to_LeftArm1.rising}" falling="${calibration.Joint_Body2_to_LeftArm1.falling}"/>
@@ -513,5 +512,5 @@
     <parent link="Link_LeftArm2"/>
     <child link="Link_LeftArm3"/>
-    <axis xyz="0 -1 0"/>
+    <axis xyz="0 1 0"/>
     <limit lower="${limits.Joint_LeftArm2_to_LeftArm3.lower}" upper="${limits.Joint_LeftArm2_to_LeftArm3.upper}" effort="${limits.Joint_LeftArm2_to_LeftArm3.effort}" velocity="${limits.Joint_LeftArm2_to_LeftArm3.velocity}"/>
     <calibration rising="${calibration.Joint_LeftArm2_to_LeftArm3.rising}" falling="${calibration.Joint_LeftArm2_to_LeftArm3.falling}"/>
@@ -544,5 +543,5 @@
     <parent link="Link_LeftArm3"/>
     <child link="Link_LeftArm4"/>
-    <axis xyz="0 0 1"/>
+    <axis xyz="0 0 -1"/>
     <limit lower="${limits.Joint_LeftArm3_to_LeftArm4.lower}" upper="${limits.Joint_LeftArm3_to_LeftArm4.upper}" effort="${limits.Joint_LeftArm3_to_LeftArm4.effort}" velocity="${limits.Joint_LeftArm3_to_LeftArm4.velocity}"/>
     <calibration rising="${calibration.Joint_LeftArm3_to_LeftArm4.rising}" falling="${calibration.Joint_LeftArm3_to_LeftArm4.falling}"/>
@@ -606,5 +605,5 @@
     <parent link="Link_LeftArm5"/>
     <child link="Link_LeftArm6"/>
-    <axis xyz="0 0 1"/>
+    <axis xyz="0 0 -1"/>
     <limit lower="${limits.Joint_LeftArm5_to_LeftArm6.lower}" upper="${limits.Joint_LeftArm5_to_LeftArm6.upper}" effort="${limits.Joint_LeftArm5_to_LeftArm6.effort}" velocity="${limits.Joint_LeftArm5_to_LeftArm6.velocity}"/>
     <calibration rising="${calibration.Joint_LeftArm5_to_LeftArm6.rising}" falling="${calibration.Joint_LeftArm5_to_LeftArm6.falling}"/>
@@ -637,5 +636,5 @@
     <parent link="Link_LeftArm6"/>
     <child link="Link_LeftArm7"/>
-    <axis xyz="0 0 -1"/>
+    <axis xyz="0 0 1"/>
     <limit lower="${limits.Joint_LeftArm6_to_LeftArm7.lower}" upper="${limits.Joint_LeftArm6_to_LeftArm7.upper}" effort="${limits.Joint_LeftArm6_to_LeftArm7.effort}" velocity="${limits.Joint_LeftArm6_to_LeftArm7.velocity}"/>
     <calibration rising="${calibration.Joint_LeftArm6_to_LeftArm7.rising}" falling="${calibration.Joint_LeftArm6_to_LeftArm7.falling}"/>
@@ -745,5 +744,5 @@
     <parent link="Link_Body2"/>
     <child link="Link_RightArm1"/>
-    <axis xyz="0 0 1"/>
+    <axis xyz="0 0 -1"/>
     <limit lower="${limits.Joint_Body2_to_RightArm1.lower}" upper="${limits.Joint_Body2_to_RightArm1.upper}" effort="${limits.Joint_Body2_to_RightArm1.effort}" velocity="${limits.Joint_Body2_to_RightArm1.velocity}"/>
     <calibration rising="${calibration.Joint_Body2_to_RightArm1.rising}" falling="${calibration.Joint_Body2_to_RightArm1.falling}"/>
@@ -838,5 +837,5 @@
     <parent link="Link_RightArm3"/>
     <child link="Link_RightArm4"/>
-    <axis xyz="0 0 -1"/>
+    <axis xyz="0 0 1"/>
     <limit lower="${limits.Joint_RightArm3_to_RightArm4.lower}" upper="${limits.Joint_RightArm3_to_RightArm4.upper}" effort="${limits.Joint_RightArm3_to_RightArm4.effort}" velocity="${limits.Joint_RightArm3_to_RightArm4.velocity}"/>
     <calibration rising="${calibration.Joint_RightArm3_to_RightArm4.rising}" falling="${calibration.Joint_RightArm3_to_RightArm4.falling}"/>
@@ -869,5 +868,5 @@
     <parent link="Link_RightArm4"/>
     <child link="Link_RightArm5"/>
-    <axis xyz="0 0 1"/>
+    <axis xyz="0 0 -1"/>
     <limit lower="${limits.Joint_RightArm4_to_RightArm5.lower}" upper="${limits.Joint_RightArm4_to_RightArm5.upper}" effort="${limits.Joint_RightArm4_to_RightArm5.effort}" velocity="${limits.Joint_RightArm4_to_RightArm5.velocity}"/>
     <calibration rising="${calibration.Joint_RightArm4_to_RightArm5.rising}" falling="${calibration.Joint_RightArm4_to_RightArm5.falling}"/>
@@ -900,5 +899,5 @@
     <parent link="Link_RightArm5"/>
     <child link="Link_RightArm6"/>
-    <axis xyz="0 0 -1"/>
+    <axis xyz="0 0 1"/>
     <limit lower="${limits.Joint_RightArm5_to_RightArm6.lower}" upper="${limits.Joint_RightArm5_to_RightArm6.upper}" effort="${limits.Joint_RightArm5_to_RightArm6.effort}" velocity="${limits.Joint_RightArm5_to_RightArm6.velocity}"/>
     <calibration rising="${calibration.Joint_RightArm5_to_RightArm6.rising}" falling="${calibration.Joint_RightArm5_to_RightArm6.falling}"/>

File: src/ylr1d_mid_control/urdf/ylr1d_mid.xacro (robot description, xacro)
@@ -8,5 +8,5 @@
   <!-- ============================================ -->
   <xacro:macro name="ylr1d" params="prefix">
-  <link name="${prefix}Link_Base">
+<link name="${prefix}Link_Base">
     <inertial>
       <origin xyz="0.037265 0.00025041 0.20252" rpy="0 0 0"/>
@@ -156,5 +156,5 @@
     <parent link="Link_LFWheelF"/>
     <child link="Link_LFWheel"/>
-    <axis xyz="0 0 1"/>
+    <axis xyz="0 0 -1"/>
     <calibration rising="${calibration.Joint_LFWheelF_to_LFWheel.rising}" falling="${calibration.Joint_LFWheelF_to_LFWheel.falling}"/>
     <dynamics damping="${dynamics.Joint_LFWheelF_to_LFWheel.damping}" friction="${dynamics.Joint_LFWheelF_to_LFWheel.friction}"/>
@@ -278,6 +278,5 @@
     <parent link="Link_LBWheelF"/>
     <child link="Link_LBWheel"/>
-    <axis xyz="0 0 1"/>
-    <limit lower="${limits.Joint_LBWheelF_to_LBWheel.lower}" upper="${limits.Joint_LBWheelF_to_LBWheel.upper}" effort="${limits.Joint_LBWheelF_to_LBWheel.effort}" velocity="${limits.Joint_LBWheelF_to_LBWheel.velocity}"/>
+    <axis xyz="0 0 -1"/>
     <calibration rising="${calibration.Joint_LBWheelF_to_LBWheel.rising}" falling="${calibration.Joint_LBWheelF_to_LBWheel.falling}"/>
     <dynamics damping="${dynamics.Joint_LBWheelF_to_LBWheel.damping}" friction="${dynamics.Joint_LBWheelF_to_LBWheel.friction}"/>
@@ -448,5 +447,5 @@
     <parent link="Link_Body2"/>
     <child link="Link_LeftArm1"/>
-    <axis xyz="0 0 -1"/>
+    <axis xyz="0 0 1"/>
     <limit lower="${limits.Joint_Body2_to_LeftArm1.lower}" upper="${limits.Joint_Body2_to_LeftArm1.upper}" effort="${limits.Joint_Body2_to_LeftArm1.effort}" velocity="${limits.Joint_Body2_to_LeftArm1.velocity}"/>
     <calibration rising="${calibration.Joint_Body2_to_LeftArm1.rising}" falling="${calibration.Joint_Body2_to_LeftArm1.falling}"/>
@@ -510,5 +509,5 @@
     <parent link="Link_LeftArm2"/>
     <child link="Link_LeftArm3"/>
-    <axis xyz="0 -1 0"/>
+    <axis xyz="0 1 0"/>
     <limit lower="${limits.Joint_LeftArm2_to_LeftArm3.lower}" upper="${limits.Joint_LeftArm2_to_LeftArm3.upper}" effort="${limits.Joint_LeftArm2_to_LeftArm3.effort}" velocity="${limits.Joint_LeftArm2_to_LeftArm3.velocity}"/>
     <calibration rising="${calibration.Joint_LeftArm2_to_LeftArm3.rising}" falling="${calibration.Joint_LeftArm2_to_LeftArm3.falling}"/>
@@ -541,5 +540,5 @@
     <parent link="Link_LeftArm3"/>
     <child link="Link_LeftArm4"/>
-    <axis xyz="0 0 1"/>
+    <axis xyz="0 0 -1"/>
     <limit lower="${limits.Joint_LeftArm3_to_LeftArm4.lower}" upper="${limits.Joint_LeftArm3_to_LeftArm4.upper}" effort="${limits.Joint_LeftArm3_to_LeftArm4.effort}" velocity="${limits.Joint_LeftArm3_to_LeftArm4.velocity}"/>
     <calibration rising="${calibration.Joint_LeftArm3_to_LeftArm4.rising}" falling="${calibration.Joint_LeftArm3_to_LeftArm4.falling}"/>
@@ -603,5 +602,5 @@
     <parent link="Link_LeftArm5"/>
     <child link="Link_LeftArm6"/>
-    <axis xyz="0 0 1"/>
+    <axis xyz="0 0 -1"/>
     <limit lower="${limits.Joint_LeftArm5_to_LeftArm6.lower}" upper="${limits.Joint_LeftArm5_to_LeftArm6.upper}" effort="${limits.Joint_LeftArm5_to_LeftArm6.effort}" velocity="${limits.Joint_LeftArm5_to_LeftArm6.velocity}"/>
     <calibration rising="${calibration.Joint_LeftArm5_to_LeftArm6.rising}" falling="${calibration.Joint_LeftArm5_to_LeftArm6.falling}"/>
@@ -634,5 +633,5 @@
     <parent link="Link_LeftArm6"/>
     <child link="Link_LeftArm7"/>
-    <axis xyz="0 0 -1"/>
+    <axis xyz="0 0 1"/>
     <limit lower="${limits.Joint_LeftArm6_to_LeftArm7.lower}" upper="${limits.Joint_LeftArm6_to_LeftArm7.upper}" effort="${limits.Joint_LeftArm6_to_LeftArm7.effort}" velocity="${limits.Joint_LeftArm6_to_LeftArm7.velocity}"/>
     <calibration rising="${calibration.Joint_LeftArm6_to_LeftArm7.rising}" falling="${calibration.Joint_LeftArm6_to_LeftArm7.falling}"/>
@@ -742,5 +741,5 @@
     <parent link="Link_Body2"/>
     <child link="Link_RightArm1"/>
-    <axis xyz="0 0 1"/>
+    <axis xyz="0 0 -1"/>
     <limit lower="${limits.Joint_Body2_to_RightArm1.lower}" upper="${limits.Joint_Body2_to_RightArm1.upper}" effort="${limits.Joint_Body2_to_RightArm1.effort}" velocity="${limits.Joint_Body2_to_RightArm1.velocity}"/>
     <calibration rising="${calibration.Joint_Body2_to_RightArm1.rising}" falling="${calibration.Joint_Body2_to_RightArm1.falling}"/>
@@ -835,5 +834,5 @@
     <parent link="Link_RightArm3"/>
     <child link="Link_RightArm4"/>
-    <axis xyz="0 0 -1"/>
+    <axis xyz="0 0 1"/>
     <limit lower="${limits.Joint_RightArm3_to_RightArm4.lower}" upper="${limits.Joint_RightArm3_to_RightArm4.upper}" effort="${limits.Joint_RightArm3_to_RightArm4.effort}" velocity="${limits.Joint_RightArm3_to_RightArm4.velocity}"/>
     <calibration rising="${calibration.Joint_RightArm3_to_RightArm4.rising}" falling="${calibration.Joint_RightArm3_to_RightArm4.falling}"/>
@@ -866,5 +865,5 @@
     <parent link="Link_RightArm4"/>
     <child link="Link_RightArm5"/>
-    <axis xyz="0 0 1"/>
+    <axis xyz="0 0 -1"/>
     <limit lower="${limits.Joint_RightArm4_to_RightArm5.lower}" upper="${limits.Joint_RightArm4_to_RightArm5.upper}" effort="${limits.Joint_RightArm4_to_RightArm5.effort}" velocity="${limits.Joint_RightArm4_to_RightArm5.velocity}"/>
     <calibration rising="${calibration.Joint_RightArm4_to_RightArm5.rising}" falling="${calibration.Joint_RightArm4_to_RightArm5.falling}"/>
@@ -897,5 +896,5 @@
     <parent link="Link_RightArm5"/>
     <child link="Link_RightArm6"/>
-    <axis xyz="0 0 -1"/>
+    <axis xyz="0 0 1"/>
     <limit lower="${limits.Joint_RightArm5_to_RightArm6.lower}" upper="${limits.Joint_RightArm5_to_RightArm6.upper}" effort="${limits.Joint_RightArm5_to_RightArm6.effort}" velocity="${limits.Joint_RightArm5_to_RightArm6.velocity}"/>
     <calibration rising="${calibration.Joint_RightArm5_to_RightArm6.rising}" falling="${calibration.Joint_RightArm5_to_RightArm6.falling}"/>
@@ -1522,5 +1521,5 @@
     </sensor>
   </gazebo>
-  <gazebo>
+    <gazebo>
     <visualise_children>true</visualise_children>
   </gazebo>
