Commit message: update the description package

File: src/ylr1d_description/urdf/ylr1d.urdf (robot description, URDF)
Before this commit: robot ylr1d, 40 links, 39 joints
Joints:
- joint Joint_Body2_to_LeftArm1: axis 0 0 -1 -> 0 0 1
- joint Joint_Body2_to_RightArm1: axis 0 0 1 -> 0 0 -1
- joint Joint_LBWheelF_to_LBWheel: axis 0 0 1 -> 0 0 -1
- joint Joint_LFWheelF_to_LFWheel: axis 0 0 1 -> 0 0 -1
- joint Joint_LeftArm1_to_LeftArm2: limit lower=-1.57 upper=1.83 effort=1000.0 velocity=2.83 -> lower=-1.83 upper=1.83 effort=1000.0 velocity=2.83
- joint Joint_LeftArm2_to_LeftArm3: axis 0 -1 0 -> 0 1 0
- joint Joint_LeftArm3_to_LeftArm4: axis 0 0 1 -> 0 0 -1
- joint Joint_LeftArm5_to_LeftArm6: axis 0 0 1 -> 0 0 -1
- joint Joint_LeftArm6_to_LeftArm7: axis 0 0 -1 -> 0 0 1
- joint Joint_RightArm1_to_RightArm2: limit lower=-1.57 upper=1.83 effort=1000.0 velocity=2.83 -> lower=-1.83 upper=1.83 effort=1000.0 velocity=2.83
- joint Joint_RightArm3_to_RightArm4: axis 0 0 -1 -> 0 0 1
- joint Joint_RightArm4_to_RightArm5: axis 0 0 1 -> 0 0 -1
- joint Joint_RightArm5_to_RightArm6: axis 0 0 -1 -> 0 0 1

File: src/ylr1d_description/urdf/ylr1d.xacro (robot description, xacro)
@@ -1,14 +1,40 @@
 <?xml version="1.0" encoding="utf-8"?>
-<robot xmlns:xacro="http://wiki.ros.org/xacro"
-       name="ylr1d">
+<robot xmlns:xacro="http://wiki.ros.org/xacro" name="ylr1d">
+  <!-- ============================================ -->
+  <!-- DESCRIPTION PACKAGE MODEL                     -->
+  <!-- This file is a copy of ylr1d_mid.xacro from  -->
+  <!-- ylr1d_mid_control, kept identical so that    -->
+  <!-- ylr1d_description can be used to display the  -->
+  <!-- robot in RViz2 and Gazebo.                    -->
+  <!--                                               -->
+  <!-- Contents:                                    -->
+  <!--  - Link/joint kinematics & inertia,          -->
+  <!--    parameterized from config YAML files      -->
+  <!--    (links/colors/limits/scale/calibration/   -->
+  <!--    dynamics) via launch mappings             -->
+  <!--  - Gazebo sensor plugins (cameras, radar,    -->
+  <!--    IMU, ultrasonic)                          -->
+  <!--  - ros2_control <ros2_control> and <gazebo>  -->
+  <!--    blocks defining control interfaces        -->
+  <!--                                               -->
+  <!-- The placeholder ${controllers_yaml_path} is  -->
+  <!-- substituted by the launch file at runtime     -->
+  <!-- with the path to config/controllers.yaml.    -->
+  <!-- ============================================ -->
   <!-- ============================================ -->
   <!-- YAML config values (links.yaml, colors.yaml,  -->
   <!-- limits.yaml, scale.yaml) are passed via xacro -->
   <!-- mappings from the launch file at runtime.     -->
-  <!-- Edit those YAML files under config/ to tune   -->
-  <!-- physical properties without touching the      -->
-  <!-- model file itself.                            -->
   <!-- ============================================ -->
   <xacro:macro name="ylr1d" params="prefix">
+<!-- 添加空的虚拟连接 -->
+<!--
+<link name="${prefix}base_footprint" />
+<joint name="${prefix}base_footprint_joint" type="fixed">
+    <origin xyz="0 0 0.3" rpy="0 0 0" />
+    <parent link="${prefix}base_footprint" />
+    <child link="${prefix}Link_Base" />
+</joint>
+-->
 <link name="${prefix}Link_Base">
     <inertial>
@@ -1094,5 +1120,642 @@
     <dynamics damping="${dynamics.Joint_Base_to_RBUltrasonicSensor.damping}" friction="${dynamics.Joint_Base_to_RBUltrasonicSensor.friction}"/>
   </joint>
+    <gazebo reference="${prefix}Link_GlobalCameraSensor">
+    <sensor type="camera" name="rgb_camera">
+      <always_on>true</always_on>
+      <update_rate>30</update_rate>
+      <topic>/global_camera/rgb/image_raw</topic>
+      <frame_name>${prefix}Link_GlobalCameraSensor</frame_name>
+      <camera>
+        <horizontal_fov>1.047</horizontal_fov>
+        <image>
+          <width>1920</width>
+          <height>1080</height>
+          <format>R8G8B8</format>
+        </image>
+        <clip>
+          <near>0.1</near>
+          <far>100.0</far>
+        </clip>
+      </camera>
+      <plugin name="global_camera_rgb_camera_plugin" filename="libgazebo_ros_camera.so">
+        <camera_name>global_camera/rgb</camera_name>
+        <cameraName>global_camera/rgb</cameraName>
+        <image_topic_name>image_raw</image_topic_name>
+        <imageTopicName>image_raw</imageTopicName>
+        <camera_info_topic_name>camera_info</camera_info_topic_name>
+        <cameraInfoTopicName>camera_info</cameraInfoTopicName>
+        <frame_name>${prefix}Link_GlobalCameraSensor</frame_name>
+        <frameName>${prefix}Link_GlobalCameraSensor</frameName>
+      </plugin>
+    </sensor>
+    <sensor type="depth" name="depth_camera">
+      <always_on>true</always_on>
+      <update_rate>30</update_rate>
+      <topic>/global_camera/depth/image_raw</topic>
+      <frame_name>${prefix}Link_GlobalCameraSensor</frame_name>
+      <camera>
+        <horizontal_fov>1.047</horizontal_fov>
+        <image>
+          <width>640</width>
+          <height>480</height>
+          <format>R8G8B8</format>
+        </image>
+        <clip>
+          <near>0.2</near>
+          <far>4.0</far>
+        </clip>
+      </camera>
+      <plugin name="global_camera_depth_camera_plugin" filename="libgazebo_ros_camera.so">
+        <camera_name>global_camera/depth</camera_name>
+        <cameraName>global_camera/depth</cameraName>
+        <image_topic_name>image_raw</image_topic_name>
+        <imageTopicName>image_raw</imageTopicName>
+        <camera_info_topic_name>camera_info</camera_info_topic_name>
+        <cameraInfoTopicName>camera_info</cameraInfoTopicName>
+        <point_cloud_topic_name>points</point_cloud_topic_name>
+        <pointCloudTopicName>points</pointCloudTopicName>
+        <frame_name>${prefix}Link_GlobalCameraSensor</frame_name>
+        <frameName>${prefix}Link_GlobalCameraSensor</frameName>
+      </plugin>
+    </sensor>
+    <sensor type="camera" name="infrared_camera">
+      <always_on>true</always_on>
+      <update_rate>15</update_rate>
+      <topic>/global_camera/infrared/image_raw</topic>
+      <frame_name>${prefix}Link_GlobalCameraSensor</frame_name>
+      <camera>
+        <horizontal_fov>1.047</horizontal_fov>
+        <image>
+          <width>640</width>
+          <height>480</height>
+          <format>R8G8B8</format>
+        </image>
+        <clip>
+          <near>0.1</near>
+          <far>10.0</far>
+        </clip>
+      </camera>
+      <plugin name="global_camera_infrared_camera_plugin" filename="libgazebo_ros_camera.so">
+        <camera_name>global_camera/infrared</camera_name>
+        <cameraName>global_camera/infrared</cameraName>
+        <image_topic_name>image_raw</image_topic_name>
+        <imageTopicName>image_raw</imageTopicName>
+        <camera_info_topic_name>camera_info</camera_info_topic_name>
+        <cameraInfoTopicName>camera_info</cameraInfoTopicName>
+        <frame_name>${prefix}Link_GlobalCameraSensor</frame_name>
+        <frameName>${prefix}Link_GlobalCameraSensor</frameName>
+      </plugin>
+    </sensor>
+  </gazebo>
+  <gazebo reference="${prefix}Link_LeftCameraSensor">
+    <sensor type="camera" name="rgb_camera">
+      <always_on>true</always_on>
+      <update_rate>30</update_rate>
+      <topic>/left_camera/rgb/image_raw</topic>
+      <frame_name>${prefix}Link_LeftCameraSensor</frame_name>
+      <camera>
+        <horizontal_fov>1.047</horizontal_fov>
+        <image>
+          <width>1920</width>
+          <height>1080</height>
+          <format>R8G8B8</format>
+        </image>
+        <clip>
+          <near>0.1</near>
+          <far>100.0</far>
+        </clip>
+      </camera>
+      <plugin name="left_camera_rgb_camera_plugin" filename="libgazebo_ros_camera.so">
+        <camera_name>left_camera/rgb</camera_name>
+        <cameraName>left_camera/rgb</cameraName>
+        <image_topic_name>image_raw</image_topic_name>
+        <imageTopicName>image_raw</imageTopicName>
+        <camera_info_topic_name>camera_info</camera_info_topic_name>
+        <cameraInfoTopicName>camera_info</cameraInfoTopicName>
+        <frame_name>${prefix}Link_LeftCameraSensor</frame_name>
+        <frameName>${prefix}Link_LeftCameraSensor</frameName>
+      </plugin>
+    </sensor>
+    <sensor type="depth" name="depth_camera">
+      <always_on>true</always_on>
+      <update_rate>30</update_rate>
+      <topic>/left_camera/depth/image_raw</topic>
+      <frame_name>${prefix}Link_LeftCameraSensor</frame_name>
+      <camera>
+        <horizontal_fov>1.047</horizontal_fov>
+        <image>
+          <width>640</width>
+          <height>480</height>
+          <format>R8G8B8</format>
+        </image>
+        <clip>
+          <near>0.2</near>
+          <far>4.0</far>
+        </clip>
+      </camera>
+      <plugin name="left_camera_depth_camera_plugin" filename="libgazebo_ros_camera.so">
+        <camera_name>left_camera/depth</camera_name>
+        <cameraName>left_camera/depth</cameraName>
+        <image_topic_name>image_raw</image_topic_name>
+        <imageTopicName>image_raw</imageTopicName>
+        <camera_info_topic_name>camera_info</camera_info_topic_name>
+        <cameraInfoTopicName>camera_info</cameraInfoTopicName>
+        <point_cloud_topic_name>points</point_cloud_topic_name>
+        <pointCloudTopicName>points</pointCloudTopicName>
+        <frame_name>${prefix}Link_LeftCameraSensor</frame_name>
+        <frameName>${prefix}Link_LeftCameraSensor</frameName>
+      </plugin>
+    </sensor>
+    <sensor type="camera" name="infrared_camera">
+      <always_on>true</always_on>
+      <update_rate>15</update_rate>
+      <topic>/left_camera/infrared/image_raw</topic>
+      <frame_name>${prefix}Link_LeftCameraSensor</frame_name>
+      <camera>
+        <horizontal_fov>1.047</horizontal_fov>
+        <image>
+          <width>640</width>
+          <height>480</height>
+          <format>R8G8B8</format>
+        </image>
+        <clip>
+          <near>0.1</near>
+          <far>10.0</far>
+        </clip>
+      </camera>
+      <plugin name="left_camera_infrared_camera_plugin" filename="libgazebo_ros_camera.so">
+        <camera_name>left_camera/infrared</camera_name>
+        <cameraName>left_camera/infrared</cameraName>
+        <image_topic_name>image_raw</image_topic_name>
+        <imageTopicName>image_raw</imageTopicName>
+        <camera_info_topic_name>camera_info</camera_info_topic_name>
+        <cameraInfoTopicName>camera_info</cameraInfoTopicName>
+        <frame_name>${prefix}Link_LeftCameraSensor</frame_name>
+        <frameName>${prefix}Link_LeftCameraSensor</frameName>
+      </plugin>
+    </sensor>
+  </gazebo>
+  <gazebo reference="${prefix}Link_RightCameraSensor">
+    <sensor type="camera" name="rgb_camera">
+      <always_on>true</always_on>
+      <update_rate>30</update_rate>
+      <topic>/right_camera/rgb/image_raw</topic>
+      <frame_name>${prefix}Link_RightCameraSensor</frame_name>
+      <camera>
+        <horizontal_fov>1.047</horizontal_fov>
+        <image>
+          <width>1920</width>
+          <height>1080</height>
+          <format>R8G8B8</format>
+        </image>
+        <clip>
+          <near>0.1</near>
+          <far>100.0</far>
+        </clip>
+      </camera>
+      <plugin name="right_camera_rgb_camera_plugin" filename="libgazebo_ros_camera.so">
+        <camera_name>right_camera/rgb</camera_name>
+        <cameraName>right_camera/rgb</cameraName>
+        <image_topic_name>image_raw</image_topic_name>
+        <imageTopicName>image_raw</imageTopicName>
+        <camera_info_topic_name>camera_info</camera_info_topic_name>
+        <cameraInfoTopicName>camera_info</cameraInfoTopicName>
+        <frame_name>${prefix}Link_RightCameraSensor</frame_name>
+        <frameName>${prefix}Link_RightCameraSensor</frameName>
+      </plugin>
+    </sensor>
+    <sensor type="depth" name="depth_camera">
+      <always_on>true</always_on>
+      <update_rate>30</update_rate>
+      <topic>/right_camera/depth/image_raw</topic>
+      <frame_name>${prefix}Link_RightCameraSensor</frame_name>
+      <camera>
+        <horizontal_fov>1.047</horizontal_fov>
+        <image>
+          <width>640</width>
+          <height>480</height>
+          <format>R8G8B8</format>
+        </image>
+        <clip>
+          <near>0.2</near>
+          <far>4.0</far>
+        </clip>
+      </camera>
+      <plugin name="right_camera_depth_camera_plugin" filename="libgazebo_ros_camera.so">
+        <camera_name>right_camera/depth</camera_name>
+        <cameraName>right_camera/depth</cameraName>
+        <image_topic_name>image_raw</image_topic_name>
+        <imageTopicName>image_raw</imageTopicName>
+        <camera_info_topic_name>camera_info</camera_info_topic_name>
+        <cameraInfoTopicName>camera_info</cameraInfoTopicName>
+        <point_cloud_topic_name>points</point_cloud_topic_name>
+        <pointCloudTopicName>points</pointCloudTopicName>
+        <frame_name>${prefix}Link_RightCameraSensor</frame_name>
+        <frameName>${prefix}Link_RightCameraSensor</frameName>
+      </plugin>
+    </sensor>
+    <sensor type="camera" name="infrared_camera">
+      <always_on>true</always_on>
+      <update_rate>15</update_rate>
+      <topic>/right_camera/infrared/image_raw</topic>
+      <frame_name>${prefix}Link_RightCameraSensor</frame_name>
+      <camera>
+        <horizontal_fov>1.047</horizontal_fov>
+        <image>
+          <width>640</width>
+          <height>480</height>
+          <format>R8G8B8</format>
+        </image>
+        <clip>
+          <near>0.1</near>
+          <far>10.0</far>
+        </clip>
+      </camera>
+      <plugin name="right_camera_infrared_camera_plugin" filename="libgazebo_ros_camera.so">
+        <camera_name>right_camera/infrared</camera_name>
+        <cameraName>right_camera/infrared</cameraName>
+        <image_topic_name>image_raw</image_topic_name>
+        <imageTopicName>image_raw</imageTopicName>
+        <camera_info_topic_name>camera_info</camera_info_topic_name>
+        <cameraInfoTopicName>camera_info</cameraInfoTopicName>
+        <frame_name>${prefix}Link_RightCameraSensor</frame_name>
+        <frameName>${prefix}Link_RightCameraSensor</frameName>
+      </plugin>
+    </sensor>
+  </gazebo>
+  <gazebo reference="${prefix}Link_RadarSensor">
+    <sensor type="ray" name="radar_sensor">
+      <always_on>true</always_on>
+      <update_rate>12</update_rate>
+      <topic>/radar/scan</topic>
+      <frame_name>${prefix}Link_RadarSensor</frame_name>
+      <ray>
+        <scan>
+          <horizontal>
+            <samples>2770</samples>
+            <resolution>1</resolution>
+            <min_angle>-3.14159</min_angle>
+            <max_angle>3.14159</max_angle>
+          </horizontal>
+        </scan>
+        <range>
+          <min>0.1</min>
+          <max>30.0</max>
+          <resolution>0.01</resolution>
+        </range>
+      </ray>
+      <noise type="gaussian">
+        <mean>0.0</mean>
+        <stddev>0.01</stddev>
+      </noise>
+      <plugin name="radar_radar_sensor_plugin" filename="libgazebo_ros_ray_sensor.so">
+        <ros>
+          <remapping>~/out:=/radar/scan</remapping>
+        </ros>
+        <output_type>sensor_msgs/LaserScan</output_type>
+      </plugin>
+    </sensor>
+  </gazebo>
+  <gazebo reference="${prefix}Link_IMUSensor">
+    <sensor type="imu" name="imu_sensor">
+      <always_on>true</always_on>
+      <update_rate>116</update_rate>
+      <topic>/imu_data</topic>
+      <frame_name>${prefix}Link_IMUSensor</frame_name>
+      <noise type="gaussian">
+        <mean>0.0</mean>
+        <stddev>0.01</stddev>
+      </noise>
+      <plugin name="imu_imu_sensor_plugin" filename="libgazebo_ros_imu_sensor.so">
+        <ros>
+          <remapping>~/out:=/imu_data</remapping>
+        </ros>
+      </plugin>
+    </sensor>
+  </gazebo>
+  <gazebo reference="${prefix}Link_LFUltrasonicSensor">
+    <sensor type="ray" name="lf_ultrasonic_sensor">
+      <always_on>true</always_on>
+      <update_rate>20</update_rate>
+      <topic>/lf_ultrasonic/range</topic>
+      <frame_name>${prefix}Link_LFUltrasonicSensor</frame_name>
+      <ray>
+        <scan>
+          <horizontal>
+            <samples>1</samples>
+            <resolution>1</resolution>
+            <min_angle>-0.5236</min_angle>
+            <max_angle>0.5236</max_angle>
+          </horizontal>
+        </scan>
+        <range>
+          <min>0.25</min>
+          <max>4.5</max>
+          <resolution>0.01</resolution>
+        </range>
+      </ray>
+      <plugin name="lf_ultrasonic_lf_ultrasonic_sensor_plugin" filename="libgazebo_ros_ray_sensor.so">
+        <ros>
+          <remapping>~/out:=/lf_ultrasonic/range</remapping>
+        </ros>
+        <output_type>sensor_msgs/LaserScan</output_type>
+      </plugin>
+    </sensor>
+  </gazebo>
+  <gazebo reference="${prefix}Link_RFUltrasonicSensor">
+    <sensor type="ray" name="rf_ultrasonic_sensor">
+      <always_on>true</always_on>
+      <update_rate>20</update_rate>
+      <topic>/rf_ultrasonic/range</topic>
+      <frame_name>${prefix}Link_RFUltrasonicSensor</frame_name>
+      <ray>
+        <scan>
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