Commit message: fix model sensor 2.0

File: src/ylr1d_description/urdf/ylr1d.xacro (robot description, xacro)
@@ -28,4 +28,12 @@
   <!-- mappings from the launch file at runtime.     -->
   <!-- ============================================ -->
+  <!-- SENSOR VISUALIZATION (diagnostic)             -->
+  <!-- ============================================ -->
+  <!-- This variant of ylr1d.xacro is used ONLY to eyeball sensor
+       position/orientation in Gazebo (see sensor_vis.launch.py). It is
+       identical to ylr1d.xacro except every sensor sets
+       <visualize>false</visualize>: ray sensors (radar + 4 ultrasonic) draw
+       their actual scan rays, cameras draw their view frustum. No physics /
+       sensor config is changed. -->
   <xacro:macro name="ylr1d" params="prefix">
 <!-- 添加空的虚拟连接 -->
@@ -444,5 +452,5 @@
   </link>
   <joint name="${prefix}Joint_Body4_to_GlobalCameraSensor" type="fixed">
-    <origin xyz="0.0566950000000047 -0.0674999999999963 0" rpy="0.000125465834204824 1.56906022137597 0.000125465645199403"/>
+    <origin xyz="0.0566950000000047 -0.0674999999999963 0" rpy="1.56906022137597 0 0.000125465645199403"/>
     <parent link="Link_Body4"/>
     <child link="Link_GlobalCameraSensor"/>
@@ -738,5 +746,5 @@
   </link>
   <joint name="${prefix}Joint_LeftArm7_to_LeftCameraSensor" type="fixed">
-    <origin xyz="-0.041999 0.00025491 0.08155" rpy="0 0 -1.5769"/>
+    <origin xyz="-0.041999 0.00025491 0.08155" rpy="3.14 -1.57686575197005 -1.5769"/>
     <parent link="Link_LeftArm7"/>
     <child link="Link_LeftCameraSensor"/>
@@ -1032,5 +1040,5 @@
   </link>
   <joint name="${prefix}Joint_RightArm7_to_RightCameraSensor" type="fixed">
-    <origin xyz="-0.0419992264026258 0.000254914269492257 0.0815499999909122" rpy="0 0 -1.57686575197005"/>
+    <origin xyz="-0.0419992264026258 0.000254914269492257 0.0815499999909122" rpy="0 -1.57686575197005 -1.57686575197005"/>
     <parent link="Link_RightArm7"/>
     <child link="Link_RightCameraSensor"/>
@@ -1047,5 +1055,5 @@
   </link>
   <joint name="${prefix}Joint_Base_to_RadarSensor" type="fixed">
-    <origin xyz="-0.237 0 0.2364" rpy="1.5708 0 -2.9674"/>
+    <origin xyz="-0.237 0 0.2364" rpy="0 0 -2.9674"/>
     <parent link="Link_Base"/>
     <child link="Link_RadarSensor"/>
@@ -1069,5 +1077,5 @@
   </link>
   <joint name="${prefix}Joint_Base_to_LFUltrasonicSensor" type="fixed">
-    <origin xyz="-0.26708 -0.18708 0.183" rpy="1.5708 0 -0.7854"/>
+    <origin xyz="-0.26708 -0.18708 0.183" rpy="1.5708 0 -2.3562"/>
     <parent link="Link_Base"/>
     <child link="Link_LFUltrasonicSensor"/>
@@ -1084,5 +1092,5 @@
   </link>
   <joint name="${prefix}Joint_Base_to_RFUltrasonicSensor" type="fixed">
-    <origin xyz="-0.26708 0.18708 0.183" rpy="1.5708 0 -2.3562"/>
+    <origin xyz="-0.26708 0.18708 0.183" rpy="1.5708 0 2.3562"/>
     <parent link="Link_Base"/>
     <child link="Link_RFUltrasonicSensor"/>
@@ -1099,5 +1107,5 @@
   </link>
   <joint name="${prefix}Joint_Base_to_LBUltrasonicSensor" type="fixed">
-    <origin xyz="0.26708 -0.18708 0.183" rpy="1.5708 0 0.7854"/>
+    <origin xyz="0.26708 -0.18708 0.183" rpy="1.5708 0 -0.7854"/>
     <parent link="Link_Base"/>
     <child link="Link_LBUltrasonicSensor"/>
@@ -1114,5 +1122,5 @@
   </link>
   <joint name="${prefix}Joint_Base_to_RBUltrasonicSensor" type="fixed">
-    <origin xyz="0.26708 0.18708 0.183" rpy="1.5708 0 2.3562"/>
+    <origin xyz="0.26708 0.18708 0.183" rpy="1.5708 0 0.7854"/>
     <parent link="Link_Base"/>
     <child link="Link_RBUltrasonicSensor"/>
@@ -1123,4 +1131,5 @@
     <gazebo reference="${prefix}Link_GlobalCameraSensor">
     <sensor type="camera" name="rgb_camera">
+      <visualize>false</visualize>
       <always_on>true</always_on>
       <update_rate>30</update_rate>
@@ -1151,4 +1160,5 @@
     </sensor>
     <sensor type="depth" name="depth_camera">
+      <visualize>false</visualize>
       <always_on>true</always_on>
       <update_rate>30</update_rate>
@@ -1181,4 +1191,5 @@
     </sensor>
     <sensor type="camera" name="infrared_camera">
+      <visualize>false</visualize>
       <always_on>true</always_on>
       <update_rate>15</update_rate>
@@ -1211,4 +1222,5 @@
   <gazebo reference="${prefix}Link_LeftCameraSensor">
     <sensor type="camera" name="rgb_camera">
+      <visualize>false</visualize>
       <always_on>true</always_on>
       <update_rate>30</update_rate>
@@ -1239,4 +1251,5 @@
     </sensor>
     <sensor type="depth" name="depth_camera">
+      <visualize>false</visualize>
       <always_on>true</always_on>
       <update_rate>30</update_rate>
@@ -1269,4 +1282,5 @@
     </sensor>
     <sensor type="camera" name="infrared_camera">
+      <visualize>false</visualize>
       <always_on>true</always_on>
       <update_rate>15</update_rate>
@@ -1299,4 +1313,5 @@
   <gazebo reference="${prefix}Link_RightCameraSensor">
     <sensor type="camera" name="rgb_camera">
+      <visualize>false</visualize>
       <always_on>true</always_on>
       <update_rate>30</update_rate>
@@ -1327,4 +1342,5 @@
     </sensor>
     <sensor type="depth" name="depth_camera">
+      <visualize>false</visualize>
       <always_on>true</always_on>
       <update_rate>30</update_rate>
@@ -1357,4 +1373,5 @@
     </sensor>
     <sensor type="camera" name="infrared_camera">
+      <visualize>false</visualize>
       <always_on>true</always_on>
       <update_rate>15</update_rate>
@@ -1387,4 +1404,5 @@
   <gazebo reference="${prefix}Link_RadarSensor">
     <sensor type="ray" name="radar_sensor">
+      <visualize>false</visualize>
       <always_on>true</always_on>
       <update_rate>12</update_rate>
@@ -1437,4 +1455,5 @@
   <gazebo reference="${prefix}Link_LFUltrasonicSensor">
     <sensor type="ray" name="lf_ultrasonic_sensor">
+      <visualize>false</visualize>
       <always_on>true</always_on>
       <update_rate>20</update_rate>
@@ -1466,4 +1485,5 @@
   <gazebo reference="${prefix}Link_RFUltrasonicSensor">
     <sensor type="ray" name="rf_ultrasonic_sensor">
+      <visualize>false</visualize>
       <always_on>true</always_on>
       <update_rate>20</update_rate>
@@ -1495,4 +1515,5 @@
   <gazebo reference="${prefix}Link_LBUltrasonicSensor">
     <sensor type="ray" name="lb_ultrasonic_sensor">
+      <visualize>false</visualize>
       <always_on>true</always_on>
       <update_rate>20</update_rate>
@@ -1524,4 +1545,5 @@
   <gazebo reference="${prefix}Link_RBUltrasonicSensor">
     <sensor type="ray" name="rb_ultrasonic_sensor">
+      <visualize>false</visualize>
       <always_on>true</always_on>
       <update_rate>20</update_rate>

File: src/ylr1d_description/urdf/ylr1d_sensor_vis.xacro (robot description, xacro)
@@ -1404,5 +1404,5 @@
   <gazebo reference="${prefix}Link_RadarSensor">
     <sensor type="ray" name="radar_sensor">
-      <!--<visualize>true</visualize>-->
+      <visualize>true</visualize>
       <always_on>true</always_on>
       <update_rate>12</update_rate>
